Commit message: Can now be opened in the moveit setup assistant

File: urdf/capra_arm.urdf.xacro (robot description, xacro)
@@ -2,13 +2,14 @@
 <robot xmlns:xacro="http://ros.org/wiki/xacro">
   <xacro:include filename="$(find robotiq_2f_140_gripper_visualization)/urdf/robotiq_arg2f_140_model_macro.xacro" />
-   <xacro:macro name="capra_arm" params="parent *origin sim">
+   <xacro:macro name="capra_arm" params="parent">
 <!-- xxxxxxxxxxxxxxxxxxxxxxxxxx Base du bras xxxxxxxxxxxxxxxxxxxxxxxxxxxxxxxx-->
      <joint name="arm_attach" type="fixed">
        <parent link="${parent}"/>
+       <origin xyz="0 0 0" rpy="0 0 0"/>
        <child link="CA_01"/>
        <dynamics damping="0.1"/>
        <limit effort="10000.0" lower="-1.49" upper="1.49" velocity="1"/>
     <!-- Utiliser l'origine specifiee dans le xacro parent -->
-       <xacro:insert_block name="origin"/>
+       <!-- <xacro:insert_block name="origin"/> -->
      </joint>
      <link name="CA_01">

File: urdf/capra_master_test.urdf.xacro (robot description, xacro)
@@ -1,37 +1,12 @@
 <?xml version="1.0"?>
-<robot xmlns:xacro="http://ros.org/wiki/xacro" name="capra_test" >
-    <!-- argument et prop placeholder -->
-    <xacro:arg name="sim" default="true"/>
-    <xacro:property name="sim" value="$(arg sim)"/>
-    <!-- urdf.xacro enfants ci dessous -->
-    <xacro:include filename="$(find capra_arm_description)/urdf/capra_arm.urdf.xacro"/>
-    <!-- Base vide -->
-    <link name="base_link">
-      <visual>
-         <geometry>
-            <box size="0.001 0.001 0.001"/>
-         </geometry>
-         <origin xyz="0. 0 0" rpy="0 0 0"/>
-         <material name="black">
-               <color rgba="0 0.1 0.1 1"/>
-         </material>
-      </visual>
-      <collision>
-         <geometry>
-            <box size="0.001 0.001 0.001"/>
-         </geometry>
-         <origin xyz="0 0 0" rpy="0 0 0"/>
-      </collision>
-      <inertial>
-        <mass value="40"/>
-          <origin xyz="0 0 0" rpy="0 0 0"/>
-          <inertia ixx = "1" ixy = "1" ixz = "1"
-                   iyy = "1" iyz = "1"
-                   izz = "1"/>
-      </inertial>
-    </link>
-    <!-- Arm -->
-    <xacro:capra_arm parent="base_link" sim="${sim}">
-        <origin xyz="0 0 0" rpy="0 0 0"/>
-    </xacro:capra_arm>
+<robot xmlns:xacro="http://ros.org/wiki/xacro" name="capra_arm">
+   <!-- argument et prop placeholder -->
+   <!-- <xacro:arg name="sim" default="true"/> -->
+   <!-- <xacro:property name="sim" value="$(arg sim)"/> -->
+   <!-- urdf.xacro enfants ci dessous -->
+   <xacro:include filename="$(find capra_arm_description)/urdf/capra_arm.urdf.xacro"/>
+   <!-- Base vide -->
+   <link name="root"/>
+   <xacro:property name="robot_root" value="root"/>
+   <xacro:capra_arm parent="${robot_root}"/>
 </robot>
