Commit message: restructured xacro.

File: urdf/capra_arm.xacro (robot description, xacro)
@@ -14,4 +14,8 @@
           <mesh filename="package://${description_pkg}/meshes/CA-01.stl"/>
         </geometry>
+        <origin xyz="0 0 0" rpy="${pi/2} 0 0"/>
+        <material name="arm_color">
+          <color rgba="0.99 0.3 0.3 1"/>
+        </material>
       </visual>
       <collision>
@@ -19,5 +23,13 @@
           <mesh filename="package://${description_pkg}/meshes/CA-01.stl"/>
         </geometry>
+        <origin xyz="0 0 0" rpy="${pi/2} 0 0"/>
       </collision>
+<!--       <inertial>
+        <mass value="0.1" />
+        <origin xyz="0.0 0.0 0.0" rpy="0 0 0"/>
+        <inertia ixx = "0.00001" ixy = "0.0" ixz = "0.0"
+                 iyy= "0.00001" iyz = "0.0"
+                 izz = "0.00001" />
+      </inertial> -->
     </link>
     <link name="${arm_id}_link1">
@@ -26,4 +38,8 @@
           <mesh filename="package://${description_pkg}/meshes/CA-02.stl"/>
         </geometry>
+        <origin xyz="0 0 0" rpy="${pi/2} 0 0"/>
+        <material name="arm_color">
+          <color rgba="0.99 0.3 0.3 1"/>
+        </material>
       </visual>
       <collision>
@@ -31,13 +47,22 @@
           <mesh filename="package://${description_pkg}/meshes/CA-02.stl"/>
         </geometry>
+        <origin xyz="0 0 0" rpy="${pi/2} 0 0"/>
       </collision>
+<!--       <inertial>
+        <mass value="0.1" />
+        <origin xyz="0.0 0.0 0.0" rpy="0 0 0"/>
+        <inertia ixx = "0.00001" ixy = "0.0" ixz = "0.0"
+                 iyy= "0.00001" iyz = "0.0"
+                 izz = "0.00001" />
+      </inertial> -->
     </link>
     <joint name="${arm_id}_joint1" type="revolute">
-      <safety_controller k_position="100.0" k_velocity="40.0" soft_lower_limit="-2.8973" soft_upper_limit="2.8973"/>
-      <origin rpy="0 0 0" xyz="0 0 0.333"/>
+      <origin xyz="0 0 0.051" rpy="0 0 0"/>
       <parent link="${arm_id}_link0"/>
       <child link="${arm_id}_link1"/>
+      <dynamics damping="0.1"/>
       <axis xyz="0 0 1"/>
-      <limit effort="87" lower="-2.8973" upper="2.8973" velocity="2.1750"/>
+      <limit effort="10000.0" lower="${-pi}" upper="${pi}" velocity="0.6"/>
+      <axis xyz="0 1 0"/>
     </joint>
     <link name="${arm_id}_link2">
@@ -54,10 +79,10 @@
     </link>
     <joint name="${arm_id}_joint2" type="revolute">
-      <safety_controller k_position="100.0" k_velocity="40.0" soft_lower_limit="-1.7628" soft_upper_limit="1.7628"/>
-      <origin rpy="${-pi/2} 0 0" xyz="0 0 0"/>
+      <origin rpy="${pi/2} 0 0" xyz="0 0 .0889"/>
       <parent link="${arm_id}_link1"/>
       <child link="${arm_id}_link2"/>
       <axis xyz="0 0 1"/>
-      <limit effort="87" lower="-1.7628" upper="1.7628" velocity="2.1750"/>
+      <limit effort="87" lower="${-pi/2}" upper="${pi/2}" velocity="2.1750"/>
+      <axis xyz="0 1 0"/>
     </joint>
     <link name="${arm_id}_link3">
@@ -74,10 +99,10 @@
     </link>
     <joint name="${arm_id}_joint3" type="revolute">
-      <safety_controller k_position="100.0" k_velocity="40.0" soft_lower_limit="-2.8973" soft_upper_limit="2.8973"/>
-      <origin rpy="${pi/2} 0 0" xyz="0 -0.316 0"/>
+      <origin rpy="0 0 ${pi/2}" xyz="0 0.3556 0"/>
       <parent link="${arm_id}_link2"/>
       <child link="${arm_id}_link3"/>
       <axis xyz="0 0 1"/>
-      <limit effort="87" lower="-2.8973" upper="2.8973" velocity="2.1750"/>
+      <limit effort="87" lower="${-pi/2}" upper="${pi/2}" velocity="2.1750"/>
+      <!-- <axis xyz="0 1 0"/> -->
     </joint>
     <link name="${arm_id}_link4">
@@ -94,10 +119,10 @@
     </link>
     <joint name="${arm_id}_joint4" type="revolute">
-      <safety_controller k_position="100.0" k_velocity="40.0" soft_lower_limit="-3.0718" soft_upper_limit="-0.0698"/>
-      <origin rpy="${pi/2} 0 0" xyz="0.0825 0 0"/>
+      <origin rpy="0 0 0" xyz="0.0889 0.047625 0"/>
       <parent link="${arm_id}_link3"/>
       <child link="${arm_id}_link4"/>
+      <axis xyz="0 1 0"/>
+      <limit effort="87" lower="${-pi}" upper="${pi}" velocity="2.1750"/>
       <axis xyz="0 0 1"/>
-      <limit effort="87" lower="-3.0718" upper="-0.0698" velocity="2.1750"/>
     </joint>
     <link name="${arm_id}_link5">
@@ -114,10 +139,10 @@
     </link>
     <joint name="${arm_id}_joint5" type="revolute">
-      <safety_controller k_position="100.0" k_velocity="40.0" soft_lower_limit="-2.8973" soft_upper_limit="2.8973"/>
-      <origin rpy="${-pi/2} 0 0" xyz="-0.0825 0.384 0"/>
+      <origin rpy="0 0 0" xyz="0 0.24765 0"/>
       <parent link="${arm_id}_link4"/>
       <child link="${arm_id}_link5"/>
       <axis xyz="0 0 1"/>
-      <limit effort="12" lower="-2.8973" upper="2.8973" velocity="2.6100"/>
+      <limit effort="10000.0" lower="${-pi/2}" upper="${pi/2}" velocity="0.57"/>
+      <axis xyz="0 1 0"/>
     </joint>
     <link name="${arm_id}_link6">
@@ -134,18 +159,16 @@
     </link>
     <joint name="${arm_id}_joint6" type="revolute">
-      <safety_controller k_position="100.0" k_velocity="40.0" soft_lower_limit="-0.0175" soft_upper_limit="3.7525"/>
-      <origin rpy="${pi/2} 0 0" xyz="0 0 0"/>
+      <origin rpy="0 ${pi/2} 0" xyz="0 0.0762 0"/>
       <parent link="${arm_id}_link5"/>
       <child link="${arm_id}_link6"/>
-      <axis xyz="0 0 1"/>
-      <limit effort="12" lower="-0.0175" upper="3.7525" velocity="2.6100"/>
+      <axis xyz="0 1 0"/>
+      <limit effort="10000.0" lower="${-pi/2}" upper="${pi/2}" velocity="0.57"/>
     </joint>
-    <link name="${arm_id}_link7"/>
-    <joint name="${arm_id}_joint7" type="fixed">
-      <origin xyz="0 0 0" rpy="0 0 0"/>
+    <!-- <link name="${arm_id}_link7"/> -->
+    <!-- <joint name="${arm_id}_joint7" type="fixed">
+      <origin xyz="0 0.09215 0" rpy="0 0 0"/>
       <parent link="${arm_id}_link6"/>
       <child link="${arm_id}_link7"/>
-      <axis xyz="0 0 0"/>
-    </joint>
+    </joint> -->
   </xacro:macro>
 </robot>

File: urdf/capra_arm_robotiq.urdf.xacro (robot description, xacro)
@@ -1,5 +1,5 @@
 <?xml version="1.0" encoding="utf-8"?>
 <robot xmlns:xacro="http://www.ros.org/wiki/xacro" name="capra_arm">
-  <xacro:include filename="$(find capra_arm_description)/urdf/panda_arm.urdf.xacro"/>
+  <xacro:include filename="$(find capra_arm_description)/urdf/capra_arm.xacro"/>
   <!-- <xacro:include filename="$(find franka_description)/robots/hand.xacro"/> -->
   <xacro:capra_arm />

Commit message: xacro clean up. ajusted  effort limit and velocity

File: urdf/capra_arm.xacro (robot description, xacro)
@@ -25,11 +25,4 @@
         <origin xyz="0 0 0" rpy="${pi/2} 0 0"/>
       </collision>
-<!--       <inertial>
-        <mass value="0.1" />
-        <origin xyz="0.0 0.0 0.0" rpy="0 0 0"/>
-        <inertia ixx = "0.00001" ixy = "0.0" ixz = "0.0"
-                 iyy= "0.00001" iyz = "0.0"
-                 izz = "0.00001" />
-      </inertial> -->
     </link>
     <link name="${arm_id}_link1">
@@ -49,11 +42,4 @@
         <origin xyz="0 0 0" rpy="${pi/2} 0 0"/>
       </collision>
-<!--       <inertial>
-        <mass value="0.1" />
-        <origin xyz="0.0 0.0 0.0" rpy="0 0 0"/>
-        <inertia ixx = "0.00001" ixy = "0.0" ixz = "0.0"
-                 iyy= "0.00001" iyz = "0.0"
-                 izz = "0.00001" />
-      </inertial> -->
     </link>
     <joint name="${arm_id}_joint1" type="revolute">
@@ -63,5 +49,5 @@
       <dynamics damping="0.1"/>
       <axis xyz="0 0 1"/>
-      <limit effort="10000.0" lower="${-pi}" upper="${pi}" velocity="0.6"/>
+      <limit effort="10000.0" lower="${-pi}" upper="${pi}" velocity="1.0"/>
       <axis xyz="0 1 0"/>
     </joint>
@@ -83,5 +69,5 @@
       <child link="${arm_id}_link2"/>
       <axis xyz="0 0 1"/>
-      <limit effort="87" lower="${-pi/2}" upper="${pi/2}" velocity="2.1750"/>
+      <limit effort="10000.0" lower="${-pi/2}" upper="${pi/2}" velocity="1.0"/>
       <axis xyz="0 1 0"/>
     </joint>
@@ -103,5 +89,5 @@
       <child link="${arm_id}_link3"/>
       <axis xyz="0 0 1"/>
-      <limit effort="87" lower="${-pi/2}" upper="${pi/2}" velocity="2.1750"/>
+      <limit effort="10000.0" lower="${-pi/2}" upper="${pi/2}" velocity="1.0"/>
       <!-- <axis xyz="0 1 0"/> -->
     </joint>
@@ -123,5 +109,5 @@
       <child link="${arm_id}_link4"/>
       <axis xyz="0 1 0"/>
-      <limit effort="87" lower="${-pi}" upper="${pi}" velocity="2.1750"/>
+      <limit effort="10000.0" lower="${-pi}" upper="${pi}" velocity="0.57"/>
       <axis xyz="0 0 1"/>
     </joint>
@@ -165,10 +151,4 @@
       <limit effort="10000.0" lower="${-pi/2}" upper="${pi/2}" velocity="0.57"/>
     </joint>
-    <!-- <link name="${arm_id}_link7"/> -->
-    <!-- <joint name="${arm_id}_joint7" type="fixed">
-      <origin xyz="0 0.09215 0" rpy="0 0 0"/>
-      <parent link="${arm_id}_link6"/>
-      <child link="${arm_id}_link7"/>
-    </joint> -->
   </xacro:macro>
 </robot>

File: urdf/capra_arm_robotiq.urdf.xacro (robot description, xacro)
@@ -5,3 +5,10 @@
   <xacro:capra_arm />
   <!-- <xacro:hand ns="panda" rpy="0 0 ${-pi/4}" connected_to="ca_link8"/> -->
+  <xacro:include filename="$(find robotiq_2f_140_gripper_visualization)/urdf/robotiq_arg2f_140_model_macro.xacro"/>
+  <xacro:robotiq_arg2f_140 prefix=""/>
+  <joint name="gripper_base" type="fixed">
+    <parent link="ca_link6"/>
+    <child link="robotiq_arg2f_base_link"/>
+    <origin xyz="0 0.09215 0" rpy="${-pi/2} ${-pi/2} 0"/>
+  </joint>
 </robot>

Commit message: Completed the arm xacro, including the robotic 2f 140

File: urdf/capra_arm.xacro (robot description, xacro)
@@ -12,14 +12,14 @@
       <visual>
         <geometry>
-          <mesh filename="package://${description_pkg}/meshes/CA-01.stl"/>
+          <mesh filename="package://${description_pkg}/meshes/visual/CA-01.stl"/>
         </geometry>
         <origin xyz="0 0 0" rpy="${pi/2} 0 0"/>
-        <material name="arm_color">
+        <!-- <material name="arm_color">
           <color rgba="0.99 0.3 0.3 1"/>
-        </material>
+        </material> -->
       </visual>
       <collision>
         <geometry>
-          <mesh filename="package://${description_pkg}/meshes/CA-01.stl"/>
+          <mesh filename="package://${description_pkg}/meshes/visual/CA-01.stl"/>
         </geometry>
         <origin xyz="0 0 0" rpy="${pi/2} 0 0"/>
@@ -29,14 +29,14 @@
       <visual>
         <geometry>
-          <mesh filename="package://${description_pkg}/meshes/CA-02.stl"/>
+          <mesh filename="package://${description_pkg}/meshes/visual/CA-02.stl"/>
         </geometry>
         <origin xyz="0 0 0" rpy="${pi/2} 0 0"/>
-        <material name="arm_color">
+        <!-- <material name="arm_color">
           <color rgba="0.99 0.3 0.3 1"/>
-        </material>
+        </material> -->
       </visual>
       <collision>
         <geometry>
-          <mesh filename="package://${description_pkg}/meshes/CA-02.stl"/>
+          <mesh filename="package://${description_pkg}/meshes/visual/CA-02.stl"/>
         </geometry>
         <origin xyz="0 0 0" rpy="${pi/2} 0 0"/>
@@ -55,10 +55,10 @@
       <visual>
         <geometry>
-          <mesh filename="package://${description_pkg}/meshes/CA-03.stl"/>
+          <mesh filename="package://${description_pkg}/meshes/visual/CA-03.stl"/>
         </geometry>
       </visual>
       <collision>
         <geometry>
-          <mesh filename="package://${description_pkg}/meshes/CA-03.stl"/>
+          <mesh filename="package://${description_pkg}/meshes/visual/CA-03.stl"/>
         </geometry>
       </collision>
@@ -75,10 +75,10 @@
       <visual>
         <geometry>
-          <mesh filename="package://${description_pkg}/meshes/CA-04.stl"/>
+          <mesh filename="package://${description_pkg}/meshes/visual/CA-04.stl"/>
         </geometry>
       </visual>
       <collision>
         <geometry>
-          <mesh filename="package://${description_pkg}/meshes/CA-04.stl"/>
+          <mesh filename="package://${description_pkg}/meshes/visual/CA-04.stl"/>
         </geometry>
       </collision>
@@ -95,10 +95,10 @@
       <visual>
         <geometry>
-          <mesh filename="package://${description_pkg}/meshes/CA-05.stl"/>
+          <mesh filename="package://${description_pkg}/meshes/visual/CA-05.stl"/>
         </geometry>
       </visual>
       <collision>
         <geometry>
-          <mesh filename="package://${description_pkg}/meshes/CA-05.stl"/>
+          <mesh filename="package://${description_pkg}/meshes/visual/CA-05.stl"/>
         </geometry>
       </collision>
@@ -115,10 +115,10 @@
       <visual>
         <geometry>
-          <mesh filename="package://${description_pkg}/meshes/CA-06.stl"/>
+          <mesh filename="package://${description_pkg}/meshes/visual/CA-06.stl"/>
         </geometry>
       </visual>
       <collision>
         <geometry>
-          <mesh filename="package://${description_pkg}/meshes/CA-06.stl"/>
+          <mesh filename="package://${description_pkg}/meshes/visual/CA-06.stl"/>
         </geometry>
       </collision>
@@ -135,19 +135,19 @@
       <visual>
         <geometry>
-          <mesh filename="package://${description_pkg}/meshes/CA-07.stl"/>
+          <mesh filename="package://${description_pkg}/meshes/visual/CA-07.stl"/>
         </geometry>
       </visual>
       <collision>
         <geometry>
-          <mesh filename="package://${description_pkg}/meshes/CA-07.stl"/>
+          <mesh filename="package://${description_pkg}/meshes/collision/CA-07.stl"/>
         </geometry>
       </collision>
     </link>
     <joint name="${arm_id}_joint6" type="revolute">
-      <origin rpy="0 ${pi/2} 0" xyz="0 0.0762 0"/>
+      <origin rpy="${pi/2} ${pi/2} 0" xyz="0 0.0762 0"/>
       <parent link="${arm_id}_link5"/>
       <child link="${arm_id}_link6"/>
-      <axis xyz="0 1 0"/>
-      <limit effort="10000.0" lower="${-pi/2}" upper="${pi/2}" velocity="0.57"/>
+      <axis xyz="0 0 1"/>
+      <limit effort="10000.0" lower="${-2*pi}" upper="${2*pi}" velocity="0.57"/>
     </joint>
   </xacro:macro>

File: urdf/capra_arm_robotiq.urdf.xacro (robot description, xacro)
@@ -10,5 +10,5 @@
     <parent link="ca_link6"/>
     <child link="robotiq_arg2f_base_link"/>
-    <origin xyz="0 0.09215 0" rpy="${-pi/2} ${-pi/2} 0"/>
+    <origin xyz="0 0 -0.09215" rpy="0 ${pi} ${pi/2}"/>
   </joint>
 </robot>

Commit message: Adjusted the stl to the actual length.

File: urdf/capra_arm.xacro (robot description, xacro)
@@ -85,5 +85,5 @@
     </link>
     <joint name="${arm_id}_joint3" type="revolute">
-      <origin rpy="0 0 ${pi/2}" xyz="0 0.3556 0"/>
+      <origin rpy="0 0 ${pi/2}" xyz="0 0.465 0"/>
       <parent link="${arm_id}_link2"/>
       <child link="${arm_id}_link3"/>
@@ -125,5 +125,5 @@
     </link>
     <joint name="${arm_id}_joint5" type="revolute">
-      <origin rpy="0 0 0" xyz="0 0.24765 0"/>
+      <origin rpy="0 0 0" xyz="0 0.265 0"/>
       <parent link="${arm_id}_link4"/>
       <child link="${arm_id}_link5"/>

Commit message: added a dummy link inside the gripper

File: urdf/capra_arm.xacro (robot description, xacro)
@@ -151,4 +151,11 @@
       <limit effort="10000.0" lower="${-2*pi}" upper="${2*pi}" velocity="0.57"/>
     </joint>
+    <link name="${arm_id}_link7">
+    </link>
+    <joint name="moveit_handle" type="fixed">
+    <parent link="${arm_id}_link6"/>
+    <child link="${arm_id}_link7"/>
+    <origin xyz="0 0 -0.26995" rpy="0 ${pi} ${pi/2}"/>
+  </joint>
   </xacro:macro>
 </robot>

Commit message: modified axis limits

File: urdf/capra_arm.xacro (robot description, xacro)
@@ -49,5 +49,5 @@
       <dynamics damping="0.1"/>
       <axis xyz="0 0 1"/>
-      <limit effort="10000.0" lower="${-pi}" upper="${pi}" velocity="1.0"/>
+      <limit effort="10000.0" lower="${-4*pi}" upper="${4*pi}" velocity="1.0"/>
       <axis xyz="0 1 0"/>
     </joint>
@@ -109,5 +109,5 @@
       <child link="${arm_id}_link4"/>
       <axis xyz="0 1 0"/>
-      <limit effort="10000.0" lower="${-pi}" upper="${pi}" velocity="0.57"/>
+      <limit effort="10000.0" lower="${-4*pi}" upper="${4*pi}" velocity="0.57"/>
       <axis xyz="0 0 1"/>
     </joint>
